File: Personal/Controller Project/Controller Project.kicad_sch (KiCad schematic)
At the start: 45 parts, among them IC1 SS49E, IC2 SS49E, SW1 SW_Push, SW10 SW_Push, SW2 SW_Push, SW3 SW_Push, SW4 SW_Push, SW5 SW_Push, SW6 SW_Push, SW7 SW_Push, SW8 SW_Push, SW9 SW_Push, U2 ESP32_DevKit_V1_DOIT

Commit message: 📝 Add the last documentation regarding the project
Other:
- moved on the sheet: IC1, IC2
Changed lines of the file:
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@@
 	(wire
 		(pts
-			(xy 107.95 50.8) (xy 116.84 50.8)
+			(xy 105.41 104.14) (xy 114.3 104.14)
 		)
 		(stroke
@@
 	(wire
 		(pts
-			(xy 107.95 38.1) (xy 116.84 38.1)
+			(xy 105.41 91.44) (xy 114.3 91.44)
 		)
 		(stroke
@@
 	)
 	(label "IC_RT"
-		(at 107.95 50.8 0)
+		(at 105.41 104.14 0)
 		(fields_autoplaced yes)
 		(effects
@@
 	)
 	(label "IC_LT"
-		(at 107.95 38.1 0)
+		(at 105.41 91.44 0)
 		(fields_autoplaced yes)
 		(effects
@@
 	(symbol
 		(lib_id "power:GND")
-		(at 116.84 35.56 270)
+		(at 114.3 88.9 270)
 		(unit 1)
 		(exclude_from_sim no)
@@
 		(fields_autoplaced yes)
 		(property "Reference" "#PWR045"
-			(at 110.49 35.56 0)
+			(at 107.95 88.9 0)
 			(effects
 				(font
@@
 		)
 		(property "Value" "GND"
-			(at 113.03 35.5599 90)
+			(at 110.49 88.8999 90)
 			(effects
 				(font
@@
 		)
 		(property "Footprint" ""
-			(at 116.84 35.56 0)
+			(at 114.3 88.9 0)
 			(effects
 				(font
@@
 		)
 		(property "Datasheet" ""
-			(at 116.84 35.56 0)
+			(at 114.3 88.9 0)
 			(effects
 				(font
@@
 		)
 		(property "Description" "Power symbol creates a global label with name \"GND\" , ground"
-			(at 116.84 35.56 0)
+			(at 114.3 88.9 0)
 			(effects
 				(font
@@
 	(symbol
 		(lib_id "power:+3.3V")
-		(at 116.84 33.02 90)
+		(at 114.3 86.36 90)
 		(unit 1)
 		(exclude_from_sim no)
@@
 		(fields_autoplaced yes)
 		(property "Reference" "#PWR047"
-			(at 120.65 33.02 0)
+			(at 118.11 86.36 0)
 			(effects
 				(font
@@
 		)
 		(property "Value" "+3.3V"
-			(at 113.03 33.0199 90)
+			(at 110.49 86.3599 90)
 			(effects
 				(font
@@
 		)
 		(property "Footprint" ""
-			(at 116.84 33.02 0)
+			(at 114.3 86.36 0)
 			(effects
 				(font
@@
 		)
 		(property "Datasheet" ""
-			(at 116.84 33.02 0)
+			(at 114.3 86.36 0)
 			(effects
 				(font
@@
 		)
 		(property "Description" "Power symbol creates a global label with name \"+3.3V\""
-			(at 116.84 33.02 0)
+			(at 114.3 86.36 0)
 			(effects
 				(font
@@
 	(symbol
 		(lib_id "power:GND")
-		(at 116.84 48.26 270)
+		(at 114.3 101.6 270)
 		(unit 1)
 		(exclude_from_sim no)
@@
 		(fields_autoplaced yes)
 		(property "Reference" "#PWR046"
-			(at 110.49 48.26 0)
+			(at 107.95 101.6 0)
 			(effects
 				(font
@@
 		)
 		(property "Value" "GND"
-			(at 113.03 48.2599 90)
+			(at 110.49 101.5999 90)
 			(effects
 				(font
@@
 		)
 		(property "Footprint" ""
-			(at 116.84 48.26 0)
+			(at 114.3 101.6 0)
 			(effects
 				(font
@@
 		)
 		(property "Datasheet" ""
-			(at 116.84 48.26 0)
+			(at 114.3 101.6 0)
 			(effects
 				(font
@@
 		)
 		(property "Description" "Power symbol creates a global label with name \"GND\" , ground"
-			(at 116.84 48.26 0)
+			(at 114.3 101.6 0)
 			(effects
 				(font
@@
 	(symbol
 		(lib_id "SS49E:SS49E")
-		(at 116.84 33.02 0)
+		(at 114.3 86.36 0)
 		(unit 1)
 		(exclude_from_sim no)
@@
 		(fields_autoplaced yes)
 		(property "Reference" "IC1"
-			(at 133.35 34.2899 0)
+			(at 130.81 87.6299 0)
 			(effects
 				(font
@@
 		)
 		(property "Value" "SS49E"
-			(at 133.35 36.8299 0)
+			(at 130.81 90.1699 0)
 			(effects
 				(font
@@
 		)
 		(property "Footprint" "SS49E:SS49E"
-			(at 133.35 127.94 0)
+			(at 130.81 181.28 0)
 			(effects
 				(font
@@
 		)
 		(property "Datasheet" "https://datasheet.datasheetarchive.com/originals/distributors/SFDatasheet-1/sf-00023632.pdf"
-			(at 133.35 227.94 0)
+			(at 130.81 281.28 0)
 			(effects
 				(font
@@
 		)
 		(property "Description" "Honeywell Ratiometric Hall Effect Sensor switching current 1.5 mA supply voltage 2.7  6.5 V dc"
-			(at 118.872 23.876 0)
+			(at 116.332 77.216 0)
 			(effects
 				(font
@@
 		)
 		(property "Height" "1.6"
-			(at 133.35 427.94 0)
+			(at 130.81 481.28 0)
 			(effects
 				(font
@@
 		)
 		(property "Mouser Part Number" "785-SS49E"
-			(at 133.35 527.94 0)
+			(at 130.81 581.28 0)
 			(effects
 				(font
@@
 		)
 		(property "Mouser Price/Stock" "https://www.mouser.co.uk/ProductDetail/Honeywell/SS49E?qs=%2Ffq2y7sSKcJBD3o5K2Vcgg%3D%3D"
-			(at 133.35 627.94 0)
+			(at 130.81 681.28 0)
 			(effects
 				(font
@@
 		)
 		(property "Manufacturer_Name" "Honeywell"
-			(at 133.35 727.94 0)
+			(at 130.81 781.28 0)
 			(effects
 				(font
@@
 		)
 		(property "Manufacturer_Part_Number" "SS49E"
-			(at 133.35 827.94 0)
+			(at 130.81 881.28 0)
 			(effects
 				(font
@@
 	(symbol
 		(lib_id "SS49E:SS49E")
-		(at 116.84 45.72 0)
+		(at 114.3 99.06 0)
 		(unit 1)
 		(exclude_from_sim no)
@@
 		(fields_autoplaced yes)
 		(property "Reference" "IC2"
-			(at 133.35 46.9899 0)
+			(at 130.81 100.3299 0)
 			(effects
 				(font
@@
 		)
 		(property "Value" "SS49E"
-			(at 133.35 49.5299 0)
+			(at 130.81 102.8699 0)
 			(effects
 				(font
@@
 		)
 		(property "Footprint" "SS49E:SS49E"
-			(at 133.35 140.64 0)
+			(at 130.81 193.98 0)
 			(effects
 				(font
@@
 		)
 		(property "Datasheet" "https://datasheet.datasheetarchive.com/originals/distributors/SFDatasheet-1/sf-00023632.pdf"
-			(at 133.35 240.64 0)
+			(at 130.81 293.98 0)
 			(effects
 				(font
@@
 		)
 		(property "Description" "Honeywell Ratiometric Hall Effect Sensor switching current 1.5 mA supply voltage 2.7  6.5 V dc"
-			(at 118.872 36.576 0)
+			(at 116.332 89.916 0)
 			(effects
 				(font
@@
 		)
 		(property "Height" "1.6"
-			(at 133.35 440.64 0)
+			(at 130.81 493.98 0)
 			(effects
 				(font
@@
 		)
 		(property "Mouser Part Number" "785-SS49E"
-			(at 133.35 540.64 0)
+			(at 130.81 593.98 0)
 			(effects
 				(font
@@
 		)
 		(property "Mouser Price/Stock" "https://www.mouser.co.uk/ProductDetail/Honeywell/SS49E?qs=%2Ffq2y7sSKcJBD3o5K2Vcgg%3D%3D"
-			(at 133.35 640.64 0)
+			(at 130.81 693.98 0)
 			(effects
 				(font
@@
 		)
 		(property "Manufacturer_Name" "Honeywell"
-			(at 133.35 740.64 0)
+			(at 130.81 793.98 0)
 			(effects
 				(font
@@
 		)
 		(property "Manufacturer_Part_Number" "SS49E"
-			(at 133.35 840.64 0)
+			(at 130.81 893.98 0)
 			(effects
 				(font
@@
 	(symbol
 		(lib_id "power:+3.3V")
-		(at 116.84 45.72 90)
+		(at 114.3 99.06 90)
 		(unit 1)
 		(exclude_from_sim no)
@@
 		(fields_autoplaced yes)
 		(property "Reference" "#PWR048"
-			(at 120.65 45.72 0)
+			(at 118.11 99.06 0)
 			(effects
 				(font
@@
 		)
 		(property "Value" "+3.3V"
-			(at 113.03 45.7199 90)
+			(at 110.49 99.0599 90)
 			(effects
 				(font
@@
 		)
 		(property "Footprint" ""
-			(at 116.84 45.72 0)
+			(at 114.3 99.06 0)
 			(effects
 				(font
@@
 		)
 		(property "Datasheet" ""
-			(at 116.84 45.72 0)
+			(at 114.3 99.06 0)
 			(effects
 				(font
@@
 		)
 		(property "Description" "Power symbol creates a global label with name \"+3.3V\""
-			(at 116.84 45.72 0)
+			(at 114.3 99.06 0)
 			(effects
 				(font
